Commit message: add visualization

File: assets/urdf/franka_description/robots/franka_panda_gripper.urdf (robot description, URDF)
Before this commit: robot panda, 16 links, 15 joints
Links:
- added link right_gripper
Joints:
- added joint right_gripper: type fixed, parent panda_hand, child right_gripper, origin xyz=0 0 0.1 rpy=0 0 3.1415926, axis 0 0 1
