Commit message: fix urdf

File: assets/urdf/franka_description/robots/franka_panda_gripper_in_hand_obj.urdf (robot description, URDF)
Before this commit: robot panda, 17 links, 16 joints
Links:
- removed link right_gripper
- added link in_hand_object_sphere1; collision sphere radius=0.066; visual sphere radius=0.066
- added link in_hand_object_sphere2; collision sphere radius=0.066; visual sphere radius=0.066
- added link in_hand_object_sphere3; collision sphere radius=0.066; visual sphere radius=0.066
- added link in_hand_object_sphere4; collision sphere radius=0.066; visual sphere radius=0.066
Joints:
- removed joint right_gripper
- added joint panda_joint_in_hand_object_sphere1: type fixed, parent panda_hand, child in_hand_object_sphere1, origin xyz=-0.05 0.0 0.13 rpy=0 0 0, axis 0 0 1
- added joint panda_joint_in_hand_object_sphere2: type fixed, parent panda_hand, child in_hand_object_sphere2, origin xyz=0.05 0.0 0.13 rpy=0 0 0, axis 0 0 1
- added joint panda_joint_in_hand_object_sphere3: type fixed, parent panda_hand, child in_hand_object_sphere3, origin xyz=-0.05 0.0 0.22 rpy=0 0 0, axis 0 0 1
- added joint panda_joint_in_hand_object_sphere4: type fixed, parent panda_hand, child in_hand_object_sphere4, origin xyz=0.05 0.0 0.22 rpy=0 0 0, axis 0 0 1

File: assets/urdf/franka_hand/robots/franka_leap_right.urdf (robot description, URDF)
Before this commit: robot panda, 30 links, 29 joints
Links:
- link dip_1: geometry collision mesh filename=meshes/leap_right_short_fingertips/dip.stl; visual mesh filename=meshes/leap_right_short_fingertips/dip.stl
- link dip_2: geometry collision mesh filename=meshes/leap_right_short_fingertips/dip.stl; visual mesh filename=meshes/leap_right_short_fingertips/dip.stl
- link dip_3: geometry collision mesh filename=meshes/leap_right_short_fingertips/dip.stl; visual mesh filename=meshes/leap_right_short_fingertips/dip.stl
- link dip_4: geometry collision mesh filename=meshes/leap_right_short_fingertips/thumb_dip.stl; visual mesh filename=meshes/leap_right_short_fingertips/thumb_dip.stl
- link fingertip_1: geometry collision mesh filename=meshes/leap_right_short_fingertips/fingertip.stl; visual mesh filename=meshes/leap_right_short_fingertips/fingertip.stl
- link fingertip_2: geometry collision mesh filename=meshes/leap_right_short_fingertips/fingertip.stl; visual mesh filename=meshes/leap_right_short_fingertips/fingertip.stl
- link fingertip_3: geometry collision mesh filename=meshes/leap_right_short_fingertips/fingertip.stl; visual mesh filename=meshes/leap_right_short_fingertips/fingertip.stl
- link fingertip_4: geometry collision mesh filename=meshes/leap_right_short_fingertips/thumb_fingertip.stl; visual mesh filename=meshes/leap_right_short_fingertips/thumb_fingertip.stl
- link mcp_joint_1: geometry collision mesh filename=meshes/leap_right_short_fingertips/mcp_joint.stl; visual mesh filename=meshes/leap_right_short_fingertips/mcp_joint.stl
- link mcp_joint_2: geometry collision mesh filename=meshes/leap_right_short_fingertips/mcp_joint.stl; visual mesh filename=meshes/leap_right_short_fingertips/mcp_joint.stl
- link mcp_joint_3: geometry collision mesh filename=meshes/leap_right_short_fingertips/mcp_joint.stl; visual mesh filename=meshes/leap_right_short_fingertips/mcp_joint.stl
- link mcp_joint_4: geometry collision mesh filename=meshes/leap_right_short_fingertips/pip.stl; visual mesh filename=meshes/leap_right_short_fingertips/pip.stl
- link palm_lower: geometry collision mesh filename=meshes/leap_right_short_fingertips/palm_lower.stl; visual mesh filename=meshes/leap_right_short_fingertips/palm_lower.stl
- link panda_link0: geometry collision mesh filename=meshes/collision/link0.obj; visual mesh filename=meshes/visual/link0.obj
- link panda_link1: geometry collision mesh filename=meshes/collision/link1.obj; visual mesh filename=meshes/visual/link1.obj
- link panda_link2: geometry collision mesh filename=meshes/collision/link2.obj; visual mesh filename=meshes/visual/link2.obj
- link panda_link3: geometry collision mesh filename=meshes/collision/link3.obj; visual mesh filename=meshes/visual/link3.obj
- link panda_link4: geometry collision mesh filename=meshes/collision/link4.obj; visual mesh filename=meshes/visual/link4.obj
- link panda_link5: geometry collision mesh filename=meshes/collision/link5.obj; visual mesh filename=meshes/visual/link5.obj
- link panda_link6: geometry collision mesh filename=meshes/collision/link6.obj; visual mesh filename=meshes/visual/link6.obj
- link panda_link7: geometry collision mesh filename=meshes/collision/link7.obj; visual mesh filename=meshes/visual/link7.obj
- link pip_1: geometry collision mesh filename=meshes/leap_right_short_fingertips/pip.stl; visual mesh filename=meshes/leap_right_short_fingertips/pip.stl
- link pip_2: geometry collision mesh filename=meshes/leap_right_short_fingertips/pip.stl; visual mesh filename=meshes/leap_right_short_fingertips/pip.stl
- link pip_3: geometry collision mesh filename=meshes/leap_right_short_fingertips/pip.stl; visual mesh filename=meshes/leap_right_short_fingertips/pip.stl
- link pip_4: geometry collision mesh filename=meshes/leap_right_short_fingertips/thumb_pip.stl; visual mesh filename=meshes/leap_right_short_fingertips/thumb_pip.stl
Joints:
- joint palm_center_joint: origin xyz=-0.03 -0.065 0 rpy=3.14159 0 -1.5707 -> xyz=0.065 -0.035 0 rpy=3.14159 0 0
