Commit message: fix meshes

File: assets/urdf/franka_hand/robots/franka_leap_right.urdf (robot description, URDF)
Before this commit: robot panda, 30 links, 29 joints
Links:
- link palm_lower: geometry collision mesh filename=meshes/leap/palm_lower.stl; visual mesh filename=meshes/leap/palm_lower.stl
