Commit message: adjust urdf and cooresponding eef initialization

File: assets/urdf/franka_hand/robots/franka_leap_right2_short_fingertips.urdf (robot description, URDF)
Before this commit: robot panda, 30 links, 29 joints
Joints:
- joint palm_center_joint: origin xyz=-0.03 -0.065 0 rpy=3.14159 0 -1.5707 -> xyz=0.065 -0.035 0 rpy=3.14159 0 0
