Commit message: fix meshes

File: assets/urdf/franka_cmd/franka_cmd_left.urdf (robot description, URDF)
Before this commit: robot franka_cmd_left, 30 links, 29 joints
Links:
- link F0J0: geometry collision mesh filename=package://franka_cmd/meshes/F0J0.stl; visual mesh filename=package://franka_cmd/meshes/F0J0.stl
- link F0J1: geometry collision mesh filename=package://franka_cmd/meshes/phalange~40mm.stl; visual mesh filename=package://franka_cmd/meshes/phalange~40mm.stl
- link F0J2: geometry collision mesh filename=package://franka_cmd/meshes/fingertip~40mm.stl; visual mesh filename=package://franka_cmd/meshes/fingertip~40mm.stl
- link F1J0: geometry collision mesh filename=package://franka_cmd/meshes/XY_roller.stl; visual mesh filename=package://franka_cmd/meshes/XY_roller.stl
- link F1J1: geometry collision mesh filename=package://franka_cmd/meshes/phalange~40mm.stl; visual mesh filename=package://franka_cmd/meshes/phalange~40mm.stl
- link F1J2: geometry collision mesh filename=package://franka_cmd/meshes/fingertip~40mm.stl; visual mesh filename=package://franka_cmd/meshes/fingertip~40mm.stl
- link F2J0: geometry collision mesh filename=package://franka_cmd/meshes/XY_roller.stl; visual mesh filename=package://franka_cmd/meshes/XY_roller.stl
- link F2J1: geometry collision mesh filename=package://franka_cmd/meshes/phalange~45mm.stl; visual mesh filename=package://franka_cmd/meshes/phalange~45mm.stl
- link F2J2: geometry collision mesh filename=package://franka_cmd/meshes/fingertip~40mm.stl; visual mesh filename=package://franka_cmd/meshes/fingertip~40mm.stl
- link F3J0: geometry collision mesh filename=package://franka_cmd/meshes/XY_roller.stl; visual mesh filename=package://franka_cmd/meshes/XY_roller.stl
- link F3J1: geometry collision mesh filename=package://franka_cmd/meshes/phalange~40mm.stl; visual mesh filename=package://franka_cmd/meshes/phalange~40mm.stl
- link F3J2: geometry collision mesh filename=package://franka_cmd/meshes/fingertip~40mm.stl; visual mesh filename=package://franka_cmd/meshes/fingertip~40mm.stl
- link F4J0: geometry collision mesh filename=package://franka_cmd/meshes/XY_roller.stl; visual mesh filename=package://franka_cmd/meshes/XY_roller.stl
- link F4J1: geometry collision mesh filename=package://franka_cmd/meshes/phalange~35mm.stl; visual mesh filename=package://franka_cmd/meshes/phalange~35mm.stl
- link F4J2: geometry collision mesh filename=package://franka_cmd/meshes/fingertip~40mm.stl; visual mesh filename=package://franka_cmd/meshes/fingertip~40mm.stl
- link palm_5_fingers: geometry collision mesh filename=package://franka_cmd/meshes/collision/palm.stl; visual mesh filename=package://franka_cmd/meshes/palm.stl

Commit message: fix asset collision mesh

File: assets/urdf/franka_cmd/franka_cmd_left.urdf (robot description, URDF)
Before this commit: robot franka_cmd_left, 30 links, 29 joints
Joints:
- joint panda_hand_joint: origin xyz=0.15 0 0.155 rpy=0 3.14159 1.5708 -> xyz=0.15 0 0.175 rpy=0 3.14159 1.5708

Commit message: fix fingertip joint

File: assets/urdf/franka_cmd/franka_cmd_left.urdf (robot description, URDF)
Before this commit: robot franka_cmd_left, 30 links, 29 joints
Joints:
- joint index_tip_joint: origin xyz=0 -0.04 0 rpy=0 0 0 -> xyz=0 0.04 0 rpy=0 0 0
- joint little_tip_joint: origin xyz=0 -0.04 0 rpy=0 0 0 -> xyz=0 0.04 0 rpy=0 0 0
- joint middle_tip_joint: origin xyz=0 -0.04 0 rpy=0 0 0 -> xyz=0 0.04 0 rpy=0 0 0
- joint ring_tip_joint: origin xyz=0 -0.04 0 rpy=0 0 0 -> xyz=0 0.04 0 rpy=0 0 0
- joint thumb_tip_joint: origin xyz=0 -0.04 0 rpy=0 0 0 -> xyz=0 0.04 0 rpy=0 0 0

File: assets/urdf/franka_cmd/franka_cmd_left_partial_thumb_colli.urdf (robot description, URDF)
Before this commit: robot franka_cmd_left, 30 links, 29 joints
Joints:
- joint index_tip_joint: origin xyz=0 -0.04 0 rpy=0 0 0 -> xyz=0 0.04 0 rpy=0 0 0
- joint little_tip_joint: origin xyz=0 -0.04 0 rpy=0 0 0 -> xyz=0 0.04 0 rpy=0 0 0
- joint middle_tip_joint: origin xyz=0 -0.04 0 rpy=0 0 0 -> xyz=0 0.04 0 rpy=0 0 0
- joint ring_tip_joint: origin xyz=0 -0.04 0 rpy=0 0 0 -> xyz=0 0.04 0 rpy=0 0 0
- joint thumb_tip_joint: origin xyz=0 -0.04 0 rpy=0 0 0 -> xyz=0 0.04 0 rpy=0 0 0

Commit message: update franka cmd asset for better collision representation

File: assets/urdf/franka_cmd/franka_cmd_left.urdf (robot description, URDF)
Before this commit: robot franka_cmd_left, 30 links, 29 joints
Links:
- link palm_5_fingers: geometry collision mesh filename=package://franka_cmd/meshes/collision/palm_2_cut.stl; visual mesh filename=package://franka_cmd/meshes/palm.stl
