Commit message: update glorbot meshes

File: assets/urdf/glorbot/glorbot.urdf (robot description, URDF)
Before this commit: robot tidybot2, 58 links, 57 joints
Links:
- link dip_1: geometry collision mesh filename=meshes/leap_right_short_fingertips/dip.stl; visual mesh filename=meshes/leap_right_short_fingertips/dip.stl
- link dip_2: geometry collision mesh filename=meshes/leap_right_short_fingertips/dip.stl; visual mesh filename=meshes/leap_right_short_fingertips/dip.stl
- link dip_3: geometry collision mesh filename=meshes/leap_right_short_fingertips/dip.stl; visual mesh filename=meshes/leap_right_short_fingertips/dip.stl
- link dip_4: geometry collision mesh filename=meshes/leap_right_short_fingertips/thumb_dip.stl; visual mesh filename=meshes/leap_right_short_fingertips/thumb_dip.stl
- link fingertip_1: geometry collision mesh filename=meshes/leap_right_short_fingertips/fingertip.stl; visual mesh filename=meshes/leap_right_short_fingertips/fingertip.stl
- link fingertip_2: geometry collision mesh filename=meshes/leap_right_short_fingertips/fingertip.stl; visual mesh filename=meshes/leap_right_short_fingertips/fingertip.stl
- link fingertip_3: geometry collision mesh filename=meshes/leap_right_short_fingertips/fingertip.stl; visual mesh filename=meshes/leap_right_short_fingertips/fingertip.stl
- link fingertip_4: geometry collision mesh filename=meshes/leap_right_short_fingertips/thumb_fingertip.stl; visual mesh filename=meshes/leap_right_short_fingertips/thumb_fingertip.stl
- link mcp_joint_1: geometry collision mesh filename=meshes/leap_right_short_fingertips/mcp_joint.stl; visual mesh filename=meshes/leap_right_short_fingertips/mcp_joint.stl
- link mcp_joint_2: geometry collision mesh filename=meshes/leap_right_short_fingertips/mcp_joint.stl; visual mesh filename=meshes/leap_right_short_fingertips/mcp_joint.stl
- link mcp_joint_3: geometry collision mesh filename=meshes/leap_right_short_fingertips/mcp_joint.stl; visual mesh filename=meshes/leap_right_short_fingertips/mcp_joint.stl
- link mcp_joint_4: geometry collision mesh filename=meshes/leap_right_short_fingertips/pip.stl; visual mesh filename=meshes/leap_right_short_fingertips/pip.stl
- link palm_lower: geometry collision mesh filename=meshes/leap_right_short_fingertips/palm_lower.stl; visual mesh filename=meshes/leap_right_short_fingertips/palm_lower.stl
- link pip_1: geometry collision mesh filename=meshes/leap_right_short_fingertips/pip.stl; visual mesh filename=meshes/leap_right_short_fingertips/pip.stl
- link pip_2: geometry collision mesh filename=meshes/leap_right_short_fingertips/pip.stl; visual mesh filename=meshes/leap_right_short_fingertips/pip.stl
- link pip_3: geometry collision mesh filename=meshes/leap_right_short_fingertips/pip.stl; visual mesh filename=meshes/leap_right_short_fingertips/pip.stl
- link pip_4: geometry collision mesh filename=meshes/leap_right_short_fingertips/thumb_pip.stl; visual mesh filename=meshes/leap_right_short_fingertips/thumb_pip.stl
