Commit message: update franka_leap assets

File: assets/franka_hand/franka_leap.urdf (robot description, URDF)
Before this commit: robot leap_hand, 22 links, 21 joints
Links:
- added link panda_link0; collision mesh filename=meshes/franka/collision/link0.obj; visual mesh filename=meshes/franka/visual/link0.dae
- added link panda_link1; collision mesh filename=meshes/franka/collision/link1.obj; visual mesh filename=meshes/franka/visual/link1.dae
- added link panda_link2; collision mesh filename=meshes/franka/collision/link2.obj; visual mesh filename=meshes/franka/visual/link2.dae
- added link panda_link3; collision mesh filename=meshes/franka/collision/link3.obj; visual mesh filename=meshes/franka/visual/link3.dae
- added link panda_link4; collision mesh filename=meshes/franka/collision/link4.obj; visual mesh filename=meshes/franka/visual/link4.dae
- added link panda_link5; collision mesh filename=meshes/franka/collision/link5.obj; visual mesh filename=meshes/franka/visual/link5.dae
- added link panda_link6; collision mesh filename=meshes/franka/collision/link6.obj; visual mesh filename=meshes/franka/visual/link6.dae
- added link panda_link7; collision mesh filename=meshes/franka/collision/link7.obj; visual mesh filename=meshes/franka/visual/link7.dae
- link dip_1: geometry collision box size=0.014 0.02 0.004; collision box size=0.014 0.02 0.004
- link dip_2: geometry collision box size=0.014 0.02 0.004; collision box size=0.014 0.02 0.004
- link dip_3: geometry collision box size=0.014 0.02 0.004; collision box size=0.014 0.02 0.004
- link dip_4: geometry collision box size=0.01 0.024 0.018; collision box size=0.014 0.02 0.004
- link fingertip_1: geometry collision box size=0.014 0.022 0.004; collision box size=0.014 0.022 0.004
- link fingertip_2: geometry collision box size=0.014 0.022 0.004; collision box size=0.014 0.022 0.004
- link fingertip_3: geometry collision box size=0.014 0.022 0.004; collision box size=0.014 0.022 0.004
- link fingertip_4: geometry collision box size=0.008 0.024 0.018; collision box size=0.02 0.004 0.03
- link mcp_1: geometry collision box size=0.014 0.02 0.004; collision box size=0.014 0.02 0.004
- link mcp_2: geometry collision box size=0.014 0.02 0.004; collision box size=0.014 0.02 0.004
- link mcp_3: geometry collision box size=0.014 0.02 0.004; collision box size=0.014 0.02 0.004
- link palm_lower: geometry collision box size=0.004 0.036 0.034; collision box size=0.01 0.12 0.02
- link pip_1: geometry collision box size=0.034 0.026 0.022; visual mesh filename=meshes/leap/visual/pip.obj
- link pip_2: geometry collision box size=0.034 0.026 0.022; visual mesh filename=meshes/leap/visual/pip.obj
- link pip_3: geometry collision box size=0.034 0.026 0.022; visual mesh filename=meshes/leap/visual/pip.obj
- link pip_4: geometry collision box size=0.014 0.004 0.02; collision box size=0.014 0.004 0.02
- link thumb_temp_base: geometry collision box size=0.034 0.026 0.022; visual mesh filename=meshes/leap/visual/pip.obj
Joints:
- added joint panda_hand_joint: type fixed, parent panda_link7, child palm_center, origin xyz=0 0 0.115 rpy=0 0 1.57079632679
- added joint panda_joint1: type revolute, parent panda_link0, child panda_link1, origin xyz=0 0 0.333 rpy=0 0 0, axis 0 0 1, limit lower=-2.8973 upper=2.8973 effort=87 velocity=2.1750
- added joint panda_joint2: type revolute, parent panda_link1, child panda_link2, origin xyz=0 0 0 rpy=-1.57079632679 0 0, axis 0 0 1, limit lower=-1.7628 upper=1.7628 effort=87 velocity=2.1750
- added joint panda_joint3: type revolute, parent panda_link2, child panda_link3, origin xyz=0 -0.316 0 rpy=1.57079632679 0 0, axis 0 0 1, limit lower=-2.8973 upper=2.8973 effort=87 velocity=2.1750
- added joint panda_joint4: type revolute, parent panda_link3, child panda_link4, origin xyz=0.0825 0 0 rpy=1.57079632679 0 0, axis 0 0 1, limit lower=-3.0718 upper=-0.0698 effort=87 velocity=2.1750
- added joint panda_joint5: type revolute, parent panda_link4, child panda_link5, origin xyz=-0.0825 0.384 0 rpy=-1.57079632679 0 0, axis 0 0 1, limit lower=-2.8973 upper=2.8973 effort=12 velocity=2.6100
- added joint panda_joint6: type revolute, parent panda_link5, child panda_link6, origin xyz=0 0 0 rpy=1.57079632679 0 0, axis 0 0 1, limit lower=-0.0175 upper=3.7525 effort=12 velocity=2.6100
- added joint panda_joint7: type revolute, parent panda_link6, child panda_link7, origin xyz=0.088 0 0 rpy=1.57079632679 0 0, axis 0 0 1, limit lower=-2.8973 upper=2.8973 effort=12 velocity=2.6100

Commit message: fix urdf axis

File: assets/franka_hand/franka_leap.urdf (robot description, URDF)
Before this commit: robot panda, 30 links, 29 joints
Joints:
- joint palm_center_joint: origin xyz=-0.03 -0.065 0 rpy=3.14159 0 -1.5707 -> xyz=0.065 -0.035 0 rpy=3.14159 0 0
- joint panda_hand_joint: origin xyz=0 0 0.115 rpy=0 0 1.57079632679 -> xyz=0 0 0.115 rpy=0 0 0
