Commit message: urdf bugfix

File: assets/franka_hand_old/franka_leap.urdf (robot description, URDF)
Before this commit: robot panda, 30 links, 29 joints
Links:
- removed link realtip_1
- removed link realtip_2
- removed link realtip_3
- removed link realtip_4
- added link index_tip_head
- added link middle_tip_head
- added link ring_tip_head
- added link thumb_tip_head
Joints:
- joint tip_joint_1: child realtip_1 -> index_tip_head
- joint tip_joint_2: child realtip_2 -> middle_tip_head
- joint tip_joint_3: child realtip_3 -> ring_tip_head
- joint tip_joint_4: child realtip_4 -> thumb_tip_head
