Commit message: update glorbot asset

File: assets/glorbot/glorbot.urdf (robot description, URDF)
Before this commit: robot tidybot2, 58 links, 57 joints
Links:
- removed link mcp_joint_1
- removed link mcp_joint_2
- removed link mcp_joint_3
- removed link mcp_joint_4
- removed link realtip_1
- removed link realtip_2
- removed link realtip_3
- removed link realtip_4
- added link index_tip_head
- added link mcp_1, mass 0.044; collision box size=0.014 0.02 0.004; collision box size=0.014 0.02 0.004
- added link mcp_2, mass 0.044; collision box size=0.014 0.02 0.004; collision box size=0.014 0.02 0.004
- added link mcp_3, mass 0.044; collision box size=0.014 0.02 0.004; collision box size=0.014 0.02 0.004
- added link middle_tip_head
- added link ring_tip_head
- added link thumb_temp_base, mass 0.032; collision box size=0.034 0.026 0.022; visual mesh filename=meshes/leap/visual/pip.obj
- added link thumb_tip_head
- link dip_1: geometry collision box size=0.014 0.02 0.004; collision box size=0.014 0.02 0.004
- link dip_2: geometry collision box size=0.014 0.02 0.004; collision box size=0.014 0.02 0.004
- link dip_3: geometry collision box size=0.014 0.02 0.004; collision box size=0.014 0.02 0.004
- link dip_4: geometry collision box size=0.01 0.024 0.018; collision box size=0.014 0.02 0.004
- link fingertip_1: geometry collision box size=0.014 0.022 0.004; collision box size=0.014 0.022 0.004
- link fingertip_2: geometry collision box size=0.014 0.022 0.004; collision box size=0.014 0.022 0.004
- link fingertip_3: geometry collision box size=0.014 0.022 0.004; collision box size=0.014 0.022 0.004
- link fingertip_4: geometry collision box size=0.008 0.024 0.018; collision box size=0.02 0.004 0.03
- link palm_lower: geometry collision box size=0.004 0.036 0.034; collision box size=0.01 0.12 0.02
- link pip_1: geometry collision box size=0.034 0.026 0.022; visual mesh filename=meshes/leap/visual/pip.obj
- link pip_2: geometry collision box size=0.034 0.026 0.022; visual mesh filename=meshes/leap/visual/pip.obj
- link pip_3: geometry collision box size=0.034 0.026 0.022; visual mesh filename=meshes/leap/visual/pip.obj
- link pip_4: geometry collision box size=0.014 0.004 0.02; collision box size=0.014 0.004 0.02
Joints:
- removed joint tip_joint_1
- removed joint tip_joint_2
- removed joint tip_joint_3
- removed joint tip_joint_4
- added joint index_tip: type fixed, parent fingertip_1, child index_tip_head, origin xyz=0 -0.048 0.015 rpy=0 0 0
- added joint middle_tip: type fixed, parent fingertip_2, child middle_tip_head, origin xyz=0 -0.048 0.015 rpy=0 0 0
- added joint ring_tip: type fixed, parent fingertip_3, child ring_tip_head, origin xyz=0 -0.048 0.015 rpy=0 0 0
- added joint thumb_tip: type fixed, parent fingertip_4, child thumb_tip_head, origin xyz=0 -0.06 -0.015 rpy=0 0 0
- joint finger_joint_0: origin xyz=-0.012200000000000007713 0.038099999999999994982 0.014500000000000000736 rpy=-1.570796326794896558 -1.0065212660796336576e-15 1.5707963267948943376 -> xyz=-0.0122 0.03810 0.01450 rpy=-1.57079 0 1.57079; parent mcp_joint_1 -> mcp_1
- joint finger_joint_1: child mcp_joint_1 -> mcp_1; origin xyz=-0.0070952496528625457958 0.023057756134899472233 -0.01872240357846021927 rpy=1.5707963267948950037 1.5707963267948945596 0 -> xyz=-0.0070 0.0230 -0.0187 rpy=1.57079 1.57079 0
- joint finger_joint_10: origin xyz=0.014999999999999971689 0.014299999999999951639 -0.012999999999999959505 rpy=1.5707963267948958919 -1.570796326794896336 0 -> xyz=0.015 0.0143 -0.013 rpy=1.57079 -1.57079 0
- joint finger_joint_11: origin xyz=9.7144514654701197287e-17 -0.036099999999999868305 0.00020000000000007511769 rpy=4.5935029425113685044e-17 -2.8730071914463799514e-16 1.5565411607615035382e-32 -> xyz=0 -0.03609 0.0002 rpy=0 0 0
- joint finger_joint_12: child mcp_joint_4 -> thumb_temp_base; origin xyz=-0.069395249652862533996 -0.0012422438651005258004 -0.021622403578460215601 rpy=-8.2381766464939424156e-17 1.5707963267948956698 0 -> xyz=-0.0693 -0.0012 -0.0216 rpy=0 1.57079 0
- joint finger_joint_13: origin xyz=-2.7755575615628913511e-17 0.014300000000000005415 -0.013000000000000011546 rpy=1.5707963267948958919 -1.570796326794896336 0 -> xyz=0 0.0143 -0.013 rpy=1.57079 -1.57079 0; parent mcp_joint_4 -> thumb_temp_base
- joint finger_joint_14: origin xyz=0 0.014499999999999966041 -0.017000000000000053263 rpy=-1.570796326794896558 1.6050198443300131245e-46 -1.9721522630516624601e-31 -> xyz=0 0.0145 -0.017 rpy=-1.57079 0 0
- joint finger_joint_15: origin xyz=-1.249000902703301108e-16 0.046599999999999863753 0.00019999999999997710581 rpy=1.5063958491491781023e-44 5.4234187233935260503e-31 3.141592653589793116 -> xyz=0 0.0466 0.0002 rpy=0 0 3.14159
- joint finger_joint_2: origin xyz=0.01499999999999996822 0.014299999999999904801 -0.012999999999999824196 rpy=1.5707963267948958919 -1.570796326794896336 0 -> xyz=0.015 0.0143 -0.013 rpy=1.57079 -1.57079 0
- joint finger_joint_3: origin xyz=-4.0880582495572692636e-09 -0.036100004210367367397 0.00020000000000007858714 rpy=4.5935029425113685044e-17 -2.8730071914463794583e-16 4.4395481053923607589e-32 -> xyz=0 -0.0361 0.0002 rpy=0 0 0
- joint finger_joint_4: origin xyz=-0.012200000000000019856 0.038099999999999981104 0.01450000000000000594 rpy=-1.570796326794896558 -1.0065212760057939085e-15 1.5707963267948943376 -> xyz=-0.0122 0.0381 0.0145 rpy=-1.57079 0 1.57079; parent mcp_joint_2 -> mcp_2
- joint finger_joint_5: child mcp_joint_2 -> mcp_2; origin xyz=-0.0070952496528625388569 -0.022392243865100525113 -0.018722403578460229678 rpy=1.570796326794896558 1.570796326794896558 0 -> xyz=-0.0071 -0.0224 -0.0187 rpy=1.57079 1.57079 0
- joint finger_joint_6: origin xyz=0.014999999999999975159 0.014300000000000000211 -0.013000000000000018485 rpy=1.5707963267948958919 -1.570796326794896336 0 -> xyz=0.015 0.0143 -0.013 rpy=1.57079 -1.57079 0
- joint finger_joint_7: origin xyz=1.0061396160665481148e-16 -0.036099999999999854428 0.00020000000000007858714 rpy=4.5935029425113654229e-17 -2.8730071914463794583e-16 1.4408183216511868558e-31 -> xyz=0 -0.0361 0.0002 rpy=0 0 0
- joint finger_joint_8: origin xyz=-0.012200000000000004244 0.038100000000000001921 0.014499999999999999001 rpy=-1.570796326794896558 -1.0065212660796360242e-15 1.5707963267948943376 -> xyz=-0.0122 0.0381 0.0145 rpy=-1.57079 0 1.57079; parent mcp_joint_3 -> mcp_3
- joint finger_joint_9: child mcp_joint_3 -> mcp_3; origin xyz=-0.0070952454426398371343 -0.067842243865100515521 -0.018722407666402932774 rpy=1.5707963267948950037 1.5707963267948945596 0 -> xyz=-0.00709 -0.0678 -0.0187 rpy=1.57079 1.57079 0
- joint palm_center_joint: origin xyz=0.065 -0.035 0 rpy=3.14159 0 0 -> xyz=-0.03 -0.065 0 rpy=3.14159 0 -1.5707
- joint panda_hand_joint: origin xyz=0 0 0.115 rpy=0 0 0 -> xyz=0 0 0.115 rpy=0 0 1.57079632679

Commit message: fix joint limit

File: assets/glorbot/glorbot.urdf (robot description, URDF)
Before this commit: robot tidybot2, 58 links, 57 joints
Joints:
- joint x5_joint1: limit lower=-10 upper=10 effort=100 velocity=1000 -> lower=-3.14 upper=2.618 effort=100 velocity=1000
