Commit message: update

File: assets/glorbot/glorbot_90shift.urdf (robot description, URDF)
Before this commit: robot tidybot2, 58 links, 57 joints
Links:
- link mcp_1: geometry collision box size=0.014 0.02 0.004; collision box size=0.014 0.02 0.004
- link mcp_2: geometry collision box size=0.014 0.02 0.004; collision box size=0.014 0.02 0.004
